Commit message: Added a xacro file for the below horizon config of the ouster

File: ouster_description/urdf/OS1-128-BH.urdf.xacro (robot description, xacro)
@@ -1,6 +1,6 @@
 <?xml version="1.0"?>
-<robot xmlns:xacro="http://www.ros.org/wiki/xacro" name="OS1-128">
+<robot xmlns:xacro="http://www.ros.org/wiki/xacro" name="OS1-128-BH">
   <xacro:property name="M_PI" value="3.1415926535897931" />
-  <xacro:macro name="OS1-128" params="*origin parent:=base_link name:=os1_sensor topic_points:=/os1_cloud_node/points topic_imu:=/os1_cloud_node/imu hz:=10 lasers:=128 samples:=512 min_range:=0.3 max_range:=120.0 noise:=0.008 min_angle:=-${M_PI} max_angle:=${M_PI} lidar_link:=os1_lidar imu_link:=os1_imu vfov_min:=-.19 vfov_max:=.19">
+  <xacro:macro name="OS1-128-BH" params="*origin parent:=base_link name:=os1_sensor topic_points:=/os1_cloud_node/points topic_imu:=/os1_cloud_node/imu hz:=10 lasers:=128 samples:=512 min_range:=0.3 max_range:=120.0 noise:=0.008 min_angle:=-${M_PI} max_angle:=${M_PI} lidar_link:=os1_lidar imu_link:=os1_imu vfov_min:=-0.19 vfov_max:=.0">
     <joint name="${name}_mount_joint" type="fixed">
       <xacro:insert_block name="origin" />
